File: rev1/rgbpad.kicad_pcb (KiCad board)
At the start: 2 copper layers, 100 x 100 mm, 17 parts, among them P1 CONN_GPIO, P2 CONN_SWD, SW1 SW_PUSH_2X2, SW2 SW_PUSH_2X2, SW3 SW_PUSH_2X2, SW4 SW_PUSH_2X2, SW5 SW_PUSH_RST, U1 STM32F030C8Tx

Commit message: Schematic done. PCB left to do.
Parts:
- added P3: CONN_01X06_RIGHT, Pin_Headers:Pin_Header_Angled_1x06, F.Cu at (197.1, 90.1)
- added P4: CONN_01X06_BOTTOM, Pin_Headers:Pin_Header_Angled_1x06, F.Cu at (216.4, 69.2)
- added P5: CONN_01X08_DEBUG, Pin_Headers:Pin_Header_Angled_1x08, F.Cu at (175.6, 69.2)
- added U10: APA102, assets:APA102, F.Cu at (185.7, 123.2)
- added U11: APA102, assets:APA102, F.Cu at (180.5, 123.2)
- added U12: APA102, assets:APA102, F.Cu at (175.3, 123.2)
- added U13: APA102, assets:APA102, F.Cu at (185.7, 114.6)
- added U14: APA102, assets:APA102, F.Cu at (180.5, 114.6)
- added U15: APA102, assets:APA102, F.Cu at (175.3, 114.6)
- added U16: APA102, assets:APA102, F.Cu at (170.1, 123.2)
- added U17: APA102, assets:APA102, F.Cu at (170.1, 114.6)
- added U2: APA102, assets:APA102, F.Cu at (206.5, 123.2)
- added U3: APA102, assets:APA102, F.Cu at (206.5, 114.6)
- added U4: APA102, assets:APA102, F.Cu at (201.3, 123.2)
- added U5: APA102, assets:APA102, F.Cu at (196.1, 123.2)
- added U6: APA102, assets:APA102, F.Cu at (190.9, 123.2)
- added U7: APA102, assets:APA102, F.Cu at (201.3, 114.6)
- added U8: APA102, assets:APA102, F.Cu at (196.1, 114.6)
- added U9: APA102, assets:APA102, F.Cu at (190.9, 114.6)
- C5: value 4u7 -> 100n
- C6: value 100n -> 4u7
- P1: value CONN_GPIO -> CONN_01X06_TOP; footprint Pin_Headers:Pin_Header_Straight_2x08 -> Socket_Strips:Socket_Strip_Angled_1x06
- P2: value CONN_SWD -> CONN_01X06_LEFT; footprint Pin_Headers:Pin_Header_Straight_1x05 -> Socket_Strips:Socket_Strip_Angled_1x06
- moved C1 172.3 mm to (253.4, 94.0)
- moved JP1 169.9 mm to (239.2, 104.3), turned to 0 degrees
- moved SW5 168.2 mm to (241.5, 94.6)
- moved C5 163.6 mm to (248.7, 105.8)
- moved C6 163.4 mm to (244.5, 101.1)
- moved C3 162.1 mm to (253.0, 105.8)
- moved C4 152.4 mm to (253.5, 99.9)
- moved C2 151.7 mm to (249.1, 94.0)
- moved R1 105.8 mm to (249.1, 99.9), turned to 0 degrees
- moved D1 104.0 mm to (244.0, 106.6)
- moved U1 90.9 mm to (183.2, 144.8), turned to 0 degrees
- moved P1 69.9 mm to (193.3, 68.9), turned to 0 degrees
- moved P2 53.6 mm to (174.8, 94.9), turned to 0 degrees
Connections:
- C1 pad 2: +3V3 -> /STM32 controller/NRST
- C6 pad 2: /STM32 controller/NRST -> +3V3
- P1 pad 1: /STM32 controller/PB14 -> /STM32 controller/NINT
- P1 pad 2: /STM32 controller/PB15 -> /STM32 controller/I2C_SDA
- P1 pad 3: /STM32 controller/PA8 -> /STM32 controller/I2C_SCL
- P1 pad 4: /STM32 controller/PA9 -> +3V3
- P1 pad 5: /STM32 controller/PA10 -> +5V
- P1 pad 6: /STM32 controller/PA11 -> GND
- P2 pad 1: +3V3 -> GND
- P2 pad 2: /STM32 controller/PA14 -> +5V
- P2 pad 3: GND -> +3V3
- P2 pad 4: /STM32 controller/PA13 -> /STM32 controller/I2C_SCL
- P2 pad 5: /STM32 controller/NRST -> /STM32 controller/I2C_SDA
- U1 pad 20: /STM32 controller/BTN11 -> /STM32 controller/PB2
- U1 pad 21: /STM32 controller/BTN13 -> /STM32 controller/BTN11
- U1 pad 22: /STM32 controller/BTN14 -> /STM32 controller/BTN12
- U1 pad 25: /STM32 controller/BTN15 -> /STM32 controller/BTN13
- U1 pad 26: /STM32 controller/BTN16 -> /STM32 controller/BTN14
- U1 pad 27: /STM32 controller/PB14 -> /STM32 controller/BTN15
- U1 pad 28: /STM32 controller/PB15 -> /STM32 controller/BTN16
- U1 pad 34: /STM32 controller/PA13 -> /STM32 controller/SYS_SWDIO
- U1 pad 37: /STM32 controller/PA14 -> /4x4_LED/DIN
- U1 pad 38: /STM32 controller/PA15 -> /4x4_LED/CIN
- U1 pad 41: /STM32 controller/PB5 -> /STM32 controller/NINT
- U1 pad 42: /STM32 controller/PB6 -> /STM32 controller/USART_TX
- U1 pad 43: /STM32 controller/PB7 -> /STM32 controller/USART_RX
- U1 pad 45: /STM32 controller/PB8 -> /STM32 controller/I2C_SCL
- U1 pad 46: /STM32 controller/BTN12 -> /STM32 controller/I2C_SDA
Routing:
- net /STM32 controller/BTN15: track 101.1 -> 0.00 mm
- net /STM32 controller/BTN9: track 96.7 -> 0.00 mm
- net /STM32 controller/BTN16: track 87.8 -> 0.00 mm
- net /STM32 controller/BTN10: track 74.8 -> 0.00 mm
- net /STM32 controller/BTN1: track 74.6 -> 0.00 mm
- net /STM32 controller/BTN3: track 69.5 -> 0.00 mm
- net /STM32 controller/BTN13: track 55.7 -> 0.00 mm
- net /STM32 controller/BTN4: track 49.5 -> 0.00 mm
- net /STM32 controller/BTN2: track 49.1 -> 0.00 mm
- net /STM32 controller/PA14: track 45.5 -> 0.00 mm
- net /STM32 controller/PA13: track 41.5 -> 0.00 mm
- net /STM32 controller/BTN5: track 38.6 -> 0.00 mm, vias 1 -> 0
- net /STM32 controller/BTN7: track 33.7 -> 0.00 mm
- net /STM32 controller/NRST: track 27.8 -> 0.00 mm, vias 1 -> 0
- net /STM32 controller/PB14: track 23.6 -> 0.00 mm
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
Commit message: This won't be easy. Or beautiful.
Parts:
- C1, C2, C3, C4, C5, C6: footprint Capacitors_SMD:C_0603_HandSoldering -> Capacitors_SMD:C_0603
- JP1: footprint Pin_Headers:Pin_Header_Straight_1x02 -> Pin_Headers:Pin_Header_Angled_1x02
- P5: value CONN_01X08_DEBUG -> CONN_01X07_DEBUG; footprint Pin_Headers:Pin_Header_Angled_1x08 -> Pin_Headers:Pin_Header_Angled_1x07
- R1: footprint Resistors_SMD:R_0603_HandSoldering -> Resistors_SMD:R_0603
- U10, U11, U12, U13, U14, U15, U16, U17, U2, U3, U4, U5, U6, U7, U8, U9: moved to B.Cu
- moved C2 184.2 mm to (69.4, 134.6)
- moved U2 156.3 mm to (62.5, 62.5), turned to 90 degrees
- moved U9 131.2 mm to (62.5, 87.5), turned to 270 degrees
- moved U3 129.9 mm to (87.5, 62.5), turned to 90 degrees
- moved JP1 129.1 mm to (136.5, 182.5)
- moved P2 125.5 mm to (52.0, 69.0), turned to 270 degrees
- moved C1 124.4 mm to (149.9, 163.0)
- moved C3 124.4 mm to (149.5, 174.8)
- moved C4 124.4 mm to (150.0, 168.9)
- moved C5 124.4 mm to (145.2, 174.8)
- moved R1 124.4 mm to (145.6, 168.9)
- moved C6 124.4 mm to (141.0, 170.1)
- moved D1 124.4 mm to (140.5, 175.6)
- moved SW5 124.4 mm to (138.0, 163.6)
- moved U10 123.7 mm to (62.5, 112.5), turned to 90 degrees
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Connections:
- P1 pad 1: /STM32 controller/NINT -> GND
- P1 pad 2: /STM32 controller/I2C_SDA -> +5V
- P1 pad 3: /STM32 controller/I2C_SCL -> +3V3
- P1 pad 4: +3V3 -> /STM32 controller/I2C_SCL
- P1 pad 5: +5V -> /STM32 controller/I2C_SDA
- P1 pad 6: GND -> /STM32 controller/NINT
- P3 pad 1: /STM32 controller/NINT -> GND
- P3 pad 2: /STM32 controller/I2C_SDA -> +5V
- P3 pad 3: /STM32 controller/I2C_SCL -> +3V3
- P3 pad 4: +3V3 -> /STM32 controller/I2C_SCL
- P3 pad 5: +5V -> /STM32 controller/I2C_SDA
- P3 pad 6: GND -> /STM32 controller/NINT
- P5 pad 1: +3V3 -> /STM32 controller/USART_TX
- P5 pad 2: /4x4_LED/DIN -> /STM32 controller/USART_RX
- P5 pad 3: GND -> /STM32 controller/NRST
- P5 pad 5: /STM32 controller/NRST -> GND
- P5 pad 6: GND -> /STM32 controller/SYS_SWDCLK
- P5 pad 7: /STM32 controller/USART_RX -> +3V3
- SW1 pad 1: GND -> /STM32 controller/BTN1
- SW1 pad 2: /STM32 controller/BTN1 -> GND
- SW1 pad 3: GND -> /STM32 controller/BTN2
- SW1 pad 4: /STM32 controller/BTN2 -> GND
- SW1 pad 5: GND -> /STM32 controller/BTN3
- SW1 pad 6: /STM32 controller/BTN3 -> GND
- SW1 pad 7: GND -> /STM32 controller/BTN4
- SW1 pad 8: /STM32 controller/BTN4 -> GND
- SW3 pad 1: GND -> /STM32 controller/BTN9
- SW3 pad 2: /STM32 controller/BTN9 -> GND
- SW3 pad 3: GND -> /STM32 controller/BTN10
- SW3 pad 4: /STM32 controller/BTN10 -> GND
- SW3 pad 5: GND -> /STM32 controller/BTN11
- SW3 pad 6: /STM32 controller/BTN11 -> GND
- SW3 pad 7: GND -> /STM32 controller/BTN12
- SW3 pad 8: /STM32 controller/BTN12 -> GND
- U1 pad 29: /STM32 controller/PA8 -> /4x4_LED/DIN
- U1 pad 30: /STM32 controller/PA9 -> /4x4_LED/CIN
- U1 pad 37: /4x4_LED/DIN -> /STM32 controller/SYS_SWDCLK
- U1 pad 38: /4x4_LED/CIN -> /STM32 controller/PA15
Routing:
- net +5V: track 0.00 -> 520.4 mm, vias 0 -> 21
- net /STM32 controller/I2C_SCL: track 0.00 -> 228.1 mm, vias 0 -> 2
- net /STM32 controller/NINT: track 0.00 -> 222.0 mm
- net /STM32 controller/I2C_SDA: track 0.00 -> 218.3 mm, vias 0 -> 2
- net +3V3: track 0.00 -> 216.7 mm, vias 0 -> 4
- net /STM32 controller/BTN6: track 0.00 -> 110.3 mm, vias 0 -> 3
- net /STM32 controller/BTN2: track 0.00 -> 103.6 mm, vias 0 -> 3
- net /STM32 controller/BTN1: track 0.00 -> 78.5 mm, vias 0 -> 3
- net /4x4_LED/CIN: track 0.00 -> 75.7 mm, vias 0 -> 1
- net /STM32 controller/BTN5: track 0.00 -> 75.5 mm, vias 0 -> 3
- net /4x4_LED/DIN: track 0.00 -> 73.5 mm, vias 0 -> 1
- net GND: track 0.00 -> 55.7 mm, vias 0 -> 13
- net /STM32 controller/SYS_SWDCLK: track 0.00 -> 53.9 mm, vias 0 -> 1
- net /STM32 controller/BTN3: track 0.00 -> 53.6 mm, vias 0 -> 1
- net /STM32 controller/BTN4: track 0.00 -> 41.2 mm, vias 0 -> 1
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Other:
- outline, holes or cut-outs redrawn
- net class +3V added: clearance 0.2032, trace_width 0.3048, via_dia 1.2, via_drill 0.6
- net class +5V added: clearance 0.2032, trace_width 0.508, via_dia 1.2, via_drill 0.6

Commit message: Guess this is it..
Parts:
- added REF**: VIA_0.6mm, assets:GND_VIA_0.6mm, F.Cu at (117.7, 75.3)
- added REF**: VIA_0.6mm, assets:GND_VIA_0.6mm, F.Cu at (130.9, 68.4)
- added REF**: VIA_0.6mm, assets:GND_VIA_0.6mm, F.Cu at (80.1, 118.8)
- added REF**: VIA_0.6mm, assets:GND_VIA_0.6mm, F.Cu at (74.2, 118.4)
- added REF**: VIA_0.6mm, assets:GND_VIA_0.6mm, B.Cu at (74.5, 102.8)
- added REF**: VIA_0.6mm, assets:GND_VIA_0.6mm, F.Cu at (59.5, 101.3)
- added REF**: VIA_0.6mm, assets:GND_VIA_0.6mm, F.Cu at (104.2, 124.7)
- added REF**: VIA_0.6mm, assets:GND_VIA_0.6mm, F.Cu at (103.0, 57.4)
- added REF**: VIA_0.6mm, assets:GND_VIA_0.6mm, F.Cu at (97.7, 57.4)
- added REF**: VIA_0.6mm, assets:GND_VIA_0.6mm, F.Cu at (132.2, 97.3)
- added REF**: VIA_0.6mm, assets:GND_VIA_0.6mm, F.Cu at (130.2, 103.5)
- added REF**: VIA_0.6mm, assets:GND_VIA_0.6mm, F.Cu at (119.0, 69.1)
- added REF**: VIA_0.6mm, assets:GND_VIA_0.6mm, F.Cu at (124.7, 128.9)
- added REF**: VIA_0.6mm, assets:GND_VIA_0.6mm, F.Cu at (135.0, 122.5)
- added REF**: VIA_0.6mm, assets:GND_VIA_0.6mm, F.Cu at (135.3, 127.9)
- added REF**: VIA_0.6mm, assets:GND_VIA_0.6mm, F.Cu at (147.1, 142.6)
- added REF**: VIA_0.6mm, assets:GND_VIA_0.6mm, F.Cu at (107.9, 147.0)
- added REF**: VIA_0.6mm, assets:GND_VIA_0.6mm, F.Cu at (104.4, 130.9)
- added REF**: VIA_0.6mm, assets:GND_VIA_0.6mm, F.Cu at (97.4, 132.2)
- added REF**: VIA_0.6mm, assets:GND_VIA_0.6mm, F.Cu at (69.5, 97.0)
- added REF**: VIA_0.6mm, assets:GND_VIA_0.6mm, F.Cu at (52.2, 59.2)
- added REF**: VIA_0.6mm, assets:GND_VIA_0.6mm, F.Cu at (59.1, 76.7)
- added REF**: VIA_0.6mm, assets:GND_VIA_0.6mm, F.Cu at (90.3, 124.8)
- added REF**: VIA_0.6mm, assets:GND_VIA_0.6mm, F.Cu at (134.3, 74.0)
- added REF**: VIA_0.6mm, assets:GND_VIA_0.6mm, F.Cu at (52.6, 90.3)
- added REF** (x2): VIA_0.6mm, assets:GND_VIA_0.6mm, F.Cu at (104.4, 119.0)
- added REF**: VIA_0.6mm, assets:GND_VIA_0.6mm, F.Cu at (124.8, 56.5)
- added REF**: VIA_0.6mm, assets:GND_VIA_0.6mm, F.Cu at (148.1, 128.4)
- added REF**: VIA_0.6mm, assets:GND_VIA_0.6mm, F.Cu at (147.7, 116.5)
- added REF**: VIA_0.6mm, assets:GND_VIA_0.6mm, F.Cu at (147.8, 89.3)
- added REF**: VIA_0.6mm, assets:GND_VIA_0.6mm, F.Cu at (132.8, 126.0)
- added REF**: VIA_0.6mm, assets:GND_VIA_0.6mm, F.Cu at (122.0, 119.7)
- added REF**: VIA_0.6mm, assets:GND_VIA_0.6mm, F.Cu at (93.2, 144.7)
- added REF**: VIA_0.6mm, assets:GND_VIA_0.6mm, F.Cu at (121.2, 126.1)
- added REF**: VIA_0.6mm, assets:GND_VIA_0.6mm, F.Cu at (122.2, 102.1)
- added REF**: VIA_0.6mm, assets:GND_VIA_0.6mm, F.Cu at (78.0, 54.5)
- added REF**: VIA_0.6mm, assets:GND_VIA_0.6mm, F.Cu at (73.2, 58.4)
- added REF**: VIA_0.6mm, assets:GND_VIA_0.6mm, F.Cu at (73.0, 68.3)
- added REF**: VIA_0.6mm, assets:GND_VIA_0.6mm, F.Cu at (97.6, 67.0)
- added REF**: VIA_0.6mm, assets:GND_VIA_0.6mm, F.Cu at (101.6, 69.2)
- added REF** (x2): VIA_0.6mm, assets:GND_VIA_0.6mm, F.Cu at (107.5, 74.8)
- added REF**: VIA_0.6mm, assets:GND_VIA_0.6mm, F.Cu at (97.2, 83.8)
- added REF**: VIA_0.6mm, assets:GND_VIA_0.6mm, B.Cu at (75.0, 115.3)
- added REF**: VIA_0.6mm, assets:GND_VIA_0.6mm, F.Cu at (93.7, 75.1)
- added REF**: VIA_0.6mm, assets:GND_VIA_0.6mm, F.Cu at (69.5, 75.5)
- added REF**: VIA_0.6mm, assets:GND_VIA_0.6mm, F.Cu at (101.5, 107.3)
- added REF**: VIA_0.6mm, assets:GND_VIA_0.6mm, F.Cu at (102.5, 105.8)
- added REF**: VIA_0.6mm, assets:GND_VIA_0.6mm, F.Cu at (112.4, 98.3)
- added REF**: VIA_0.6mm, assets:GND_VIA_0.6mm, F.Cu at (112.4, 100.2)
- added REF**: VIA_0.6mm, assets:GND_VIA_0.6mm, F.Cu at (115.5, 98.0)
- added REF**: VIA_0.6mm, assets:GND_VIA_0.6mm, F.Cu at (109.0, 98.5)
- added REF**: VIA_0.6mm, assets:GND_VIA_0.6mm, F.Cu at (83.0, 98.5)
- added REF**: VIA_0.6mm, assets:GND_VIA_0.6mm, F.Cu at (84.5, 96.8)
- added REF**: VIA_0.6mm, assets:GND_VIA_0.6mm, B.Cu at (73.2, 110.4)
- added REF**: VIA_0.6mm, assets:GND_VIA_0.6mm, F.Cu at (81.6, 96.5)
- added REF**: VIA_0.6mm, assets:GND_VIA_0.6mm, F.Cu at (76.9, 80.7)
- added REF**: VIA_0.6mm, assets:GND_VIA_0.6mm, F.Cu at (75.5, 80.7)
- added REF**: VIA_0.6mm, assets:GND_VIA_0.6mm, F.Cu at (98.0, 115.3)
- added REF**: VIA_0.6mm, assets:GND_VIA_0.6mm, F.Cu at (123.0, 85.6)
- added REF**: VIA_0.6mm, assets:GND_VIA_0.6mm, F.Cu at (94.3, 100.1)
- added REF**: VIA_0.6mm, assets:GND_VIA_0.6mm, F.Cu at (53.8, 100.0)
- added REF**: VIA_0.6mm, assets:GND_VIA_0.6mm, F.Cu at (67.0, 120.7)
- added REF**: VIA_0.6mm, assets:GND_VIA_0.6mm, F.Cu at (86.9, 134.3)
- added REF**: VIA_0.6mm, assets:GND_VIA_0.6mm, F.Cu at (135.3, 71.0)
- moved JP1 98.0 mm to (55.9, 126.8), turned to 90 degrees
- moved C3 94.4 mm to (66.0, 130.9)
- moved C5 91.5 mm to (66.0, 129.1)
- moved D1 85.1 mm to (66.0, 134.5)
- moved R1 84.9 mm to (68.4, 133.7), turned to 90 degrees
- moved C4 76.2 mm to (82.9, 132.8), turned to 270 degrees
- moved C6 67.6 mm to (84.6, 132.8), turned to 270 degrees
- moved C1 65.2 mm to (86.9, 146.1), turned to 270 degrees
- moved SW5 50.8 mm to (90.5, 145.5), turned to 270 degrees
- moved C2 3.85 mm to (66.0, 132.8)
Connections:
- JP1 pad 1: /STM32 controller/BOOT0 -> GND
- JP1 pad 2: GND -> /STM32 controller/BOOT0
Routing:
- net +3V3: track 216.7 -> 319.9 mm, vias 4 -> 6
- net /STM32 controller/BTN8: track 0.00 -> 86.7 mm, vias 0 -> 3
- net GND: track 55.7 -> 141.1 mm, vias 13 -> 35
- net /STM32 controller/BTN16: track 0.00 -> 84.0 mm, vias 0 -> 1
- net /STM32 controller/BTN14: track 0.00 -> 68.3 mm, vias 0 -> 1
- net /STM32 controller/I2C_SCL: track 228.1 -> 296.0 mm, vias 2 -> 4
- net +5V: track 520.4 -> 584.7 mm, vias 21 -> 25
- net /STM32 controller/I2C_SDA: track 218.3 -> 282.1 mm, vias 2 -> 4
- net /STM32 controller/BTN11: track 0.00 -> 55.9 mm, vias 0 -> 5
- net /STM32 controller/BTN7: track 0.00 -> 54.7 mm, vias 0 -> 1
- net /STM32 controller/NINT: track 222.0 -> 276.5 mm
- net /STM32 controller/USART_TX: track 0.00 -> 45.7 mm
- net /STM32 controller/USART_RX: track 0.00 -> 40.2 mm
- net /STM32 controller/BTN15: track 0.00 -> 39.4 mm, vias 0 -> 3
- net /STM32 controller/BTN13: track 0.00 -> 33.8 mm, vias 0 -> 4
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
Commit message: New PCB layout
Parts:
- removed the REF** at (117.7, 75.3)
- removed the REF** at (130.9, 68.4)
- removed the REF** at (80.1, 118.8)
- removed the REF** at (74.2, 118.4)
- removed the REF** at (74.5, 102.8)
- removed the REF** at (59.5, 101.3)
- removed the REF** at (104.2, 124.7)
- removed the REF** at (103.0, 57.4)
- removed the REF** at (97.7, 57.4)
- removed the REF** at (132.2, 97.3)
- removed the REF** at (130.2, 103.5)
- removed the REF** at (119.0, 69.1)
- removed the REF** at (124.7, 128.9)
- removed the REF** at (135.0, 122.5)
- removed the REF** at (135.3, 127.9)
- removed the REF** at (147.1, 142.6)
- removed the REF** at (107.9, 147.0)
- removed the REF** at (104.4, 130.9)
- removed the REF** at (97.4, 132.2)
- removed the REF** at (69.5, 97.0)
- removed the REF** at (52.2, 59.2)
- removed the REF** at (59.1, 76.7)
- removed the REF** at (90.3, 124.8)
- removed the REF** at (134.3, 74.0)
- removed the REF** at (52.6, 90.3)
- removed the REF** at (104.4, 119.0) (x2)
- removed the REF** at (124.8, 56.5)
- removed the REF** at (148.1, 128.4)
- removed the REF** at (147.7, 116.5)
- removed the REF** at (147.8, 89.3)
- removed the REF** at (132.8, 126.0)
- removed the REF** at (122.0, 119.7)
- removed the REF** at (93.2, 144.7)
- removed the REF** at (121.2, 126.1)
- removed the REF** at (122.2, 102.1)
- removed the REF** at (78.0, 54.5)
- removed the REF** at (73.2, 58.4)
- removed the REF** at (73.0, 68.3)
- removed the REF** at (97.6, 67.0)
- removed the REF** at (101.6, 69.2)
- removed the REF** at (107.5, 74.8) (x2)
- removed the REF** at (97.2, 83.8)
- removed the REF** at (75.0, 115.3)
- removed the REF** at (93.7, 75.1)
- removed the REF** at (69.5, 75.5)
- removed the REF** at (101.5, 107.3)
- removed the REF** at (102.5, 105.8)
- removed the REF** at (112.4, 98.3)
- removed the REF** at (112.4, 100.2)
- removed the REF** at (115.5, 98.0)
- removed the REF** at (109.0, 98.5)
- removed the REF** at (83.0, 98.5)
- removed the REF** at (84.5, 96.8)
- removed the REF** at (73.2, 110.4)
- removed the REF** at (81.6, 96.5)
- removed the REF** at (76.9, 80.7)
- removed the REF** at (75.5, 80.7)
- removed the REF** at (98.0, 115.3)
- removed the REF** at (123.0, 85.6)
- removed the REF** at (94.3, 100.1)
- removed the REF** at (53.8, 100.0)
- removed the REF** at (67.0, 120.7)
- removed the REF** at (86.9, 134.3)
- removed the REF** at (135.3, 71.0)
- added REF**: VIA_0.6mm, assets:GND_VIA_0.6mm, F.Cu at (125.2, 132.6)
- added REF**: VIA_0.6mm, assets:GND_VIA_0.6mm, F.Cu at (114.3, 148.8)
- added REF**: VIA_0.6mm, assets:GND_VIA_0.6mm, F.Cu at (112.8, 148.8)
- added REF**: VIA_0.6mm, assets:GND_VIA_0.6mm, F.Cu at (111.0, 148.8)
- added REF**: VIA_0.6mm, assets:GND_VIA_0.6mm, F.Cu at (109.2, 148.8)
- added REF**: VIA_0.6mm, assets:GND_VIA_0.6mm, F.Cu at (106.4, 148.8)
- added REF**: VIA_0.6mm, assets:GND_VIA_0.6mm, F.Cu at (128.2, 142.1)
- added REF**: VIA_0.6mm, assets:GND_VIA_0.6mm, F.Cu at (128.0, 143.5)
- added REF**: VIA_0.6mm, assets:GND_VIA_0.6mm, F.Cu at (126.6, 143.5)
- added REF**: VIA_0.6mm, assets:GND_VIA_0.6mm, F.Cu at (148.3, 51.8)
- added REF**: VIA_0.6mm, assets:GND_VIA_0.6mm, F.Cu at (51.9, 51.8)
- added REF**: VIA_0.6mm, assets:GND_VIA_0.6mm, F.Cu at (146.8, 148.6)
- added REF**: VIA_0.6mm, assets:GND_VIA_0.6mm, F.Cu at (52.1, 148.0)
- added REF**: VIA_0.6mm, assets:GND_VIA_0.6mm, F.Cu at (134.4, 75.4)
- added REF**: VIA_0.6mm, assets:GND_VIA_0.6mm, F.Cu at (134.1, 125.2)
- added REF**: VIA_0.6mm, assets:GND_VIA_0.6mm, F.Cu at (148.1, 148.1)
- added REF**: VIA_0.6mm, assets:GND_VIA_0.6mm, F.Cu at (148.1, 146.3)
- added REF**: VIA_0.6mm, assets:GND_VIA_0.6mm, F.Cu at (146.8, 147.1)
- added REF**: VIA_0.6mm, assets:GND_VIA_0.6mm, F.Cu at (149.1, 93.2)
- added REF**: VIA_0.6mm, assets:GND_VIA_0.6mm, F.Cu at (110.2, 146.8)
- added REF**: VIA_0.6mm, assets:GND_VIA_0.6mm, F.Cu at (115.3, 146.8)
- added REF**: VIA_0.6mm, assets:GND_VIA_0.6mm, F.Cu at (113.8, 146.8)
- added REF**: VIA_0.6mm, assets:GND_VIA_0.6mm, F.Cu at (112.0, 146.8)
- C1, C2, C3, C4, C5, C6, D1, JP1, P1, P2, P3, P4, P5, R1, SW5, U1: moved to B.Cu
- SW1, SW2, SW3, SW4, U10, U11, U12, U13, U14, U15, U16, U17, U2, U3, U4, U5, U6, U7, U8, U9: moved to F.Cu
- moved C3 54.4 mm to (103.0, 90.9), turned to 270 degrees
- moved C1 44.6 mm to (87.5, 101.5), turned to 90 degrees
- moved SW5 44.1 mm to (84.9, 101.7), turned to 90 degrees
- moved C2 42.9 mm to (90.1, 97.3)
- moved P1 37.5 mm to (93.6, 52.0), turned to 0 degrees
- moved P2 37.4 mm to (54.0, 106.3), turned to 90 degrees
- moved P4 37.4 mm to (93.6, 145.9)
- moved P3 37.3 mm to (145.9, 106.3)
- moved D1 36.9 mm to (82.2, 101.4), turned to 270 degrees
- moved U1 35.6 mm to (99.8, 100.0), turned to 0 degrees
- moved SW1 35.4 mm to (75.0, 75.0)
- moved SW2 35.4 mm to (125.0, 75.0)
- moved SW4 35.4 mm to (125.0, 125.0)
- moved SW3 35.3 mm to (75.0, 125.0)
- moved P5 35.0 mm to (117.6, 146.0)
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Connections:
- JP1 pad 1: GND -> /STM32 controller/BOOT0
- JP1 pad 2: /STM32 controller/BOOT0 -> GND
- P1 pad 1: GND -> /STM32 controller/NINT
- P1 pad 2: +5V -> /STM32 controller/I2C_SDA
- P1 pad 3: +3V3 -> /STM32 controller/I2C_SCL
- P1 pad 4: /STM32 controller/I2C_SCL -> +3V3
- P1 pad 5: /STM32 controller/I2C_SDA -> +5V
- P1 pad 6: /STM32 controller/NINT -> GND
- P2 pad 1: GND -> /STM32 controller/NINT
- P2 pad 2: +5V -> /STM32 controller/I2C_SDA
- P2 pad 3: +3V3 -> /STM32 controller/I2C_SCL
- P2 pad 4: /STM32 controller/I2C_SCL -> +3V3
- P2 pad 5: /STM32 controller/I2C_SDA -> +5V
- P2 pad 6: /STM32 controller/NINT -> GND
- P3 pad 1: GND -> /STM32 controller/NINT
- P3 pad 2: +5V -> /STM32 controller/I2C_SDA
- P3 pad 3: +3V3 -> /STM32 controller/I2C_SCL
- P3 pad 4: /STM32 controller/I2C_SCL -> +3V3
- P3 pad 5: /STM32 controller/I2C_SDA -> +5V
- P3 pad 6: /STM32 controller/NINT -> GND
- P4 pad 1: GND -> /STM32 controller/NINT
- P4 pad 2: +5V -> /STM32 controller/I2C_SDA
- P4 pad 3: +3V3 -> /STM32 controller/I2C_SCL
- P4 pad 4: /STM32 controller/I2C_SCL -> +3V3
- P4 pad 5: /STM32 controller/I2C_SDA -> +5V
- P4 pad 6: /STM32 controller/NINT -> GND
- SW1 pad 5: /STM32 controller/BTN3 -> /STM32 controller/BTN5
- SW1 pad 7: /STM32 controller/BTN4 -> /STM32 controller/BTN6
- SW2 pad 1: /STM32 controller/BTN5 -> /STM32 controller/BTN3
- SW2 pad 3: /STM32 controller/BTN6 -> /STM32 controller/BTN4
- SW3 pad 5: /STM32 controller/BTN11 -> /STM32 controller/BTN13
- SW3 pad 7: /STM32 controller/BTN12 -> /STM32 controller/BTN14
- SW4 pad 1: /STM32 controller/BTN13 -> /STM32 controller/BTN11
- SW4 pad 3: /STM32 controller/BTN14 -> /STM32 controller/BTN12
Routing:
- net /STM32 controller/BTN6: track 108.4 -> 0.00 mm, vias 3 -> 0
- net /STM32 controller/BTN2: track 101.8 -> 0.00 mm, vias 3 -> 0
- net /STM32 controller/BTN8: track 86.7 -> 0.00 mm, vias 3 -> 0
- net /STM32 controller/I2C_SCL: track 296.0 -> 211.0 mm, vias 4 -> 5
- net /STM32 controller/BTN16: track 84.0 -> 0.00 mm, vias 1 -> 0
- net /4x4_LED/CIN: track 76.4 -> 0.00 mm, vias 1 -> 0
- net /STM32 controller/BTN1: track 75.5 -> 0.00 mm, vias 3 -> 0
- net /STM32 controller/BTN5: track 75.3 -> 0.00 mm, vias 3 -> 0
- net /4x4_LED/DIN: track 74.6 -> 0.00 mm, vias 1 -> 0
- net /STM32 controller/BTN14: track 68.3 -> 0.00 mm, vias 1 -> 0
- net /STM32 controller/I2C_SDA: track 282.1 -> 214.2 mm, vias 4 -> 6
- net /STM32 controller/NRST: track 32.7 -> 100.5 mm, vias 1 -> 3
- net GND: track 141.1 -> 201.6 mm, vias 35 -> 18
- net /STM32 controller/BTN7: track 54.7 -> 0.00 mm, vias 1 -> 0
- net /STM32 controller/BTN3: track 51.9 -> 0.00 mm, vias 1 -> 0
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
Commit message: Minor fixes
Parts:
- added REF**: VIA_0.6mm, assets:GND_VIA_0.6mm, F.Cu at (103.6, 118.6)
- added REF**: VIA_0.6mm, assets:GND_VIA_0.6mm, F.Cu at (84.3, 73.7)
- added REF**: VIA_0.6mm, assets:GND_VIA_0.6mm, F.Cu at (120.9, 67.8)
- added REF**: VIA_0.6mm, assets:GND_VIA_0.6mm, F.Cu at (128.8, 56.4)
- moved C2 1.95 mm to (88.1, 97.3)
- moved REF** 0.82 mm to (127.4, 143.5)
- moved REF** 0.76 mm to (128.8, 143.5)
- moved REF** 0.38 mm to (128.2, 142.5)
Routing:
- net /STM32 controller/BTN1: track 0.00 -> 75.5 mm, vias 0 -> 3
- net /STM32 controller/BTN5: track 0.00 -> 61.5 mm, vias 0 -> 5
- net /4x4_LED/CIN: track 0.00 -> 57.6 mm, vias 0 -> 3
- net /STM32 controller/BTN3: track 0.00 -> 55.8 mm, vias 0 -> 1
- net /STM32 controller/BTN4: track 0.00 -> 54.4 mm, vias 0 -> 1
- net /STM32 controller/BTN2: track 0.00 -> 51.8 mm, vias 0 -> 1
- net /STM32 controller/BTN8: track 0.00 -> 47.1 mm, vias 0 -> 2
- net /4x4_LED/DIN: track 0.00 -> 43.9 mm, vias 0 -> 2
- net /STM32 controller/BTN6: track 0.00 -> 33.7 mm, vias 0 -> 1
- net /STM32 controller/BTN7: track 0.00 -> 14.9 mm, vias 0 -> 1
- net +3V3: track 369.0 -> 369.9 mm
