File: rev1/rgbpad.kicad_pcb (KiCad board)
At the start: 2 copper layers, 100 x 100 mm, 63 parts, among them P1 CONN_01X06_TOP, P2 CONN_01X06_LEFT, P3 CONN_01X06_RIGHT, P4 CONN_01X06_BOTTOM, P5 CONN_01X07_DEBUG, SW1 SW_PUSH_2X2, SW2 SW_PUSH_2X2, SW3 SW_PUSH_2X2, SW4 SW_PUSH_2X2, SW5 SW_PUSH_RST, U1 STM32F030C8Tx, U10 APA102, U11 APA102, U12 APA102, U13 APA102, U14 APA102, U15 APA102, U16 APA102, U17 APA102, U2 APA102, U3 APA102, U4 APA102, U5 APA102, U6 APA102, U7 APA102, U8 APA102, U9 APA102

Commit message: Final commit for R1
Parts:
- removed the REF** at (114.3, 148.8)
- removed the REF** at (112.8, 148.8)
- removed the REF** at (111.0, 148.8)
- removed the REF** at (109.2, 148.8)
- removed the REF** at (106.4, 148.8)
- removed the REF** at (148.3, 51.8)
- added G***: LOGO, assets:logo_32x25mm, B.Cu at (99.5, 75.0)
- added REF**: MountingHole_3.2mm_M3, Mounting_Holes:MountingHole_3.2mm_M3, F.Cu at (52.5, 52.5)
- added REF**: VIA_0.6mm, assets:GND_VIA_0.6mm, F.Cu at (125.7, 74.9)
- added REF**: VIA_0.6mm, assets:GND_VIA_0.6mm, F.Cu at (74.9, 124.7)
- added REF**: VIA_0.6mm, assets:GND_VIA_0.6mm, F.Cu at (71.1, 123.2)
- added REF**: VIA_0.6mm, assets:GND_VIA_0.6mm, F.Cu at (96.0, 125.0)
- added REF**: VIA_0.6mm, assets:GND_VIA_0.6mm, F.Cu at (93.5, 123.2)
- added REF**: VIA_0.6mm, assets:GND_VIA_0.6mm, F.Cu at (103.4, 123.4)
- added REF**: VIA_0.6mm, assets:GND_VIA_0.6mm, F.Cu at (106.9, 124.2)
- added REF**: VIA_0.6mm, assets:GND_VIA_0.6mm, F.Cu at (69.8, 130.3)
- added REF**: VIA_0.6mm, assets:GND_VIA_0.6mm, F.Cu at (69.6, 145.5)
- added REF**: VIA_0.6mm, assets:GND_VIA_0.6mm, F.Cu at (58.0, 148.5)
- added REF**: MountingHole_3.2mm_M3, Mounting_Holes:MountingHole_3.2mm_M3, F.Cu at (147.5, 52.5)
- added REF**: VIA_0.6mm, assets:GND_VIA_0.6mm, F.Cu at (56.6, 147.1)
- added REF**: VIA_0.6mm, assets:GND_VIA_0.6mm, F.Cu at (51.5, 142.0)
- added REF**: VIA_0.6mm, assets:GND_VIA_0.6mm, F.Cu at (53.0, 143.0)
- added REF**: MountingHole_3.2mm_M3, Mounting_Holes:MountingHole_3.2mm_M3, F.Cu at (147.5, 147.5)
- added REF**: VIA_0.6mm, assets:GND_VIA_0.6mm, F.Cu at (102.4, 141.2)
- added REF**: MountingHole_3.2mm_M3, Mounting_Holes:MountingHole_3.2mm_M3, F.Cu at (52.5, 147.5)
- added REF**: VIA_0.6mm, assets:GND_VIA_0.6mm, F.Cu at (101.9, 136.4)
- added REF**: VIA_0.6mm, assets:GND_VIA_0.6mm, F.Cu at (102.9, 132.1)
- added REF**: VIA_0.6mm, assets:GND_VIA_0.6mm, F.Cu at (141.2, 97.5)
- added REF**: VIA_0.6mm, assets:GND_VIA_0.6mm, F.Cu at (134.9, 97.8)
- added REF**: VIA_0.6mm, assets:GND_VIA_0.6mm, F.Cu at (131.1, 96.5)
- moved REF** 4.84 mm to (55.1, 55.4)
- moved REF** 4.56 mm to (56.6, 148.5)
- moved REF** 4.32 mm to (146.8, 144.3)
- moved REF** 4.32 mm to (148.1, 142.0)
- moved REF** 4.32 mm to (146.8, 142.7)
- moved REF** 4.32 mm to (148.1, 143.8)
Routing:
- net /STM32 controller/BTN13: track 0.00 -> 128.0 mm, vias 0 -> 3
- net /STM32 controller/BTN14: track 0.00 -> 115.5 mm, vias 0 -> 3
- net /STM32 controller/BTN15: track 0.00 -> 83.6 mm, vias 0 -> 3
- net /4x4_LED/DIN: track 43.9 -> 115.5 mm, vias 2 -> 5
- net /STM32 controller/BTN9: track 0.00 -> 68.5 mm, vias 0 -> 3
- net /STM32 controller/BTN16: track 0.00 -> 57.7 mm, vias 0 -> 1
- net /4x4_LED/CIN: track 57.6 -> 109.4 mm, vias 3 -> 5
- net /STM32 controller/BTN12: track 0.00 -> 44.7 mm, vias 0 -> 3
- net /STM32 controller/BTN10: track 0.00 -> 27.9 mm, vias 0 -> 3
- net GND: track 201.6 -> 217.3 mm
- net /STM32 controller/NRST: track 100.5 -> 104.7 mm
- net +3V3: track 369.9 -> 365.7 mm
- net /STM32 controller/SYS_SWDIO: track 64.0 -> 66.6 mm
- net /STM32 controller/BTN2: track 51.8 -> 53.3 mm
- net /STM32 controller/BTN3: track 55.8 -> 54.6 mm
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Other:
- board text added: "*"
- board text added: "+3.3V"
- board text added: "+5V"
- board text added: "BOOT0"
- board text added: "GND"
- board text added: "RESET"
- board text added: "RGB PAD 4x4 R1 2016-07 kbeckmann"
- board text added: "SCL"
- board text added: "SDA"
- board text added: "SWDCLK"
- board text added: "SWDIO"
- board text added: "U_RX"
- board text added: "U_TX"
- board text added: "~INT~"
- board text added: "~RST~"
